File: cella_di_lievitazione_kicad/cella_di_lievitazione_kicad.kicad_sch (KiCad schematic)
At the start: 2 parts

Commit message: no message
Parts:
- removed F2: Fuse, symbol Device:Fuse
- added Q1: NMOS, symbol Simulation_SPICE:NMOS
- added R2: Heater, symbol Device:Heater
- added U1: STM32G030K6Tx, Package_QFP:LQFP-32_7x7mm_P0.8mm, symbol MCU_ST_STM32G0:STM32G030K6Tx
Connections:
- net at F1.1: now also Q1.3 (S)
- net at F1.2: now also R2.1
- new net GND: R2.2

Commit message: no message
Parts:
- removed R2: Heater, symbol Device:Heater
Other:
- added sheet Heater (heater.kicad_sch)
Changed lines of the file:
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@@
-	)
-	(symbol
-		(lib_id "Device:Heater")
-		(at 215.9 116.84 0)
-		(unit 1)
-		(exclude_from_sim no)
-		(in_bom yes)
-		(on_board yes)
-		(dnp no)
-		(fields_autoplaced yes)
-		(property "Reference" "R2"
-			(at 218.44 115.5699 0)
-			(effects
-				(font
-					(size 1.27 1.27)
-				)
-				(justify left)
-			)
-		)
-		(property "Value" "Heater"
-			(at 218.44 118.1099 0)
-			(effects
-				(font
-					(size 1.27 1.27)
-				)
-				(justify left)
-			)
-		)
-		(property "Footprint" ""
-			(at 214.122 116.84 90)
-			(effects
-				(font
-					(size 1.27 1.27)
-				)
-				(hide yes)
-			)
-		)
-		(property "Datasheet" "~"
-			(at 215.9 116.84 0)
-			(effects
-				(font
-					(size 1.27 1.27)
-				)
-				(hide yes)
-			)
-		)
-		(property "Description" "Resistive heater"
-			(at 215.9 116.84 0)
-			(effects
-				(font
-					(size 1.27 1.27)
-				)
-				(hide yes)
-			)
-		)
-		(pin "2"
-		)
-		(pin "1"
-		)
-		(instances
-			(project ""
-				(path "/23c110f9-dc10-4f3f-b23a-337251207cdc"
-					(reference "R2")
-					(unit 1)
-				)
-			)
-		)
 	)
 	(symbol
@@
 				)
 			)
+		)
+	)
+	(sheet
+		(at 190.5 50.8)
+		(size 25.4 25.4)
+		(exclude_from_sim no)
+		(in_bom yes)
+		(on_board yes)
+		(dnp no)
+		(fields_autoplaced yes)
+		(stroke
+			(width 0.1524)
+			(type solid)
+		)
+		(fill
+			(color 0 0 0 0.0000)
+		)
+		(property "Sheetname" "Heater"
+			(at 190.5 50.0884 0)
+			(effects
+				(font
+					(size 1.27 1.27)
+				)
+				(justify left bottom)
+			)
+		)
+		(property "Sheetfile" "heater.kicad_sch"
+			(at 190.5 76.7846 0)
+			(effects
+				(font
+					(size 1.27 1.27)
+				)
+				(justify left top)
+				(hide yes)
+			)
+		)
+		(pin "V_heater_N" output
+			(at 190.5 69.85 180)
+			(effects
+				(font
+					(size 1.27 1.27)
+				)
+				(justify left)
+			)
+		)
+		(pin "V_heater_P" input
+			(at 190.5 57.15 180)
+			(effects
+				(font
+					(size 1.27 1.27)
+				)
+				(justify left)
+			)
+		)
+		(instances
+			(project "cella_di_lievitazione_kicad"
+				(path "/23c110f9-dc10-4f3f-b23a-337251207cdc"
+					(page "2")
+				)
+			)

Commit message: no message
Parts:
- removed F1: Fuse, symbol Device:Fuse
- removed Q1: NMOS, symbol Simulation_SPICE:NMOS
- removed U1: STM32G030K6Tx, Package_QFP:LQFP-32_7x7mm_P0.8mm, symbol MCU_ST_STM32G0:STM32G030K6Tx
Other:
- added sheet Alimentazione (alimentazione.kicad_sch)
- added sheet uC (uC.kicad_sch)

Commit message: no message
Parts:
- added J3: Screw_Terminal_01x12, symbol Connector:Screw_Terminal_01x12
- added R12: R, symbol Device:R
Connections:
- new net NET1: J3.4 (Pin_4)
- new net USB1: J3.1 (Pin_1)
- new net USB2: J3.2 (Pin_2), R12.1
- new net USB3: J3.3 (Pin_3), R12.2
- no-connect marks 0 -> 1
