File: cella_di_lievitazione_kicad/alimentazione.kicad_sch (KiCad schematic)
At the start: 0 parts

Commit message: no message
Parts:
- added C2, C3: 1u, symbol Device:C
- added C4, C5: 100n, symbol Device:C
- added J1: Screw_Terminal_01x02, symbol Connector:Screw_Terminal_01x02
- added J2: USB_C_Receptacle_PowerOnly_24P, symbol Connector:USB_C_Receptacle_PowerOnly_24P
- added SW2: SW_Nidec_CAS-120A1, Button_Switch_SMD:Nidec_Copal_CAS-120A, symbol Switch:SW_Nidec_CAS-120A1
- added U1: CYPD3177-24LQ, Package_DFN_QFN:QFN-24-1EP_4x4mm_P0.5mm_EP2.75x2.75mm, symbol Interface_USB:CYPD3177-24LQ
Connections:
- new net: C2.1, C4.1, C5.1, U1.23 (VDDD)
- new net: U1.19 (GND), U1.22 (GND), U1.25 (GND)
- new net: C3.1, U1.24 (VCCD)
- new net: J2.A1 (GND), J2.A12 (GND), J2.B1 (GND), J2.B12 (GND)
- new net: J2.A4 (VBUS), J2.A9 (VBUS), J2.B4 (VBUS), J2.B9 (VBUS)
- new net GND: C2.2, C3.2, C4.2, C5.2

Commit message: no message
Parts:
- added F2: Fuse, symbol Device:Fuse
- added Q3: NMOS, symbol Simulation_SPICE:NMOS
Connections:
- new net: F2.1, Q3.3 (S)
Other:
- moved on the sheet: C2, C3, C4, C5

Commit message: no message
Parts:
- added R15, R16, R17, R18, R3, R4, R5, R6: R, symbol Device:R
Connections:
- net GND: now also R16.2, R18.2, R4.2, R6.2
- net at U1.1 (VBUS_MIN): now also R5.2, R6.1
- net at U1.2 (VBUS_MAX): now also R3.2, R4.1
- net at U1.5 (ISNK_COARSE): now also R15.2, R16.1
- net at U1.6 (ISNK_FINE): now also R17.2, R18.1
Other:
- note added: "VDDIO"
